File: RevA_Mecanismos/RevA_Mecanismos/RevA_Mecanismos.kicad_pcb (KiCad board)
At the start: 4 copper layers, 99.7 x 99.7 mm, 137 parts, among them IC1 MAX33040EAKA+T, J1 Conn_01x02_Socket, J10 430450224, J11 430450224, J12 Conn_01x08_Socket, J13 Conn_01x08_Socket, J14 Conn_01x02_Pin, J15 430450624, J16 Conn_01x07_Pin, J17 Conn_01x02_Pin, J18 Conn_01x02_Pin, J19 Conn_01x02_Pin, J2 PROG, J20 3557-2, J21 Conn_01x04_Pin, J22 Conn_01x04_Pin, J3 Conn_01x02_Pin, J4 430450224, J5 430450224, J6 430450224, J7 430450224, J8 3557-2, J9 3557-2, Q1 FDN335N, Q2 NDS352AP, Q3 IRF9540NSPBF, Q4 IRF9540NSPBF, Q5 IRF9540NSPBF, Q6 IRF9540NSPBF, SW1 SW_Push, U1 STM32L431RCTx, U2 R-78E3.3-1.0, U3 R-78E5.0-1.0, U4 IRF540SPBF, U5 IRF540SPBF, U6 IRF540SPBF, U7 IRF540SPBF, U8 TXB0104D, Y1 16MHz

Commit message: Corrections to component footprints in schematic design made during the development of BOM
Parts:
- J1: value Conn_01x02_Socket -> Conn_01x02_Pin
- R40: value R -> 33
Changed lines of the file:
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@@
       (sketchpadsonfab false)
       (subtractmaskfromsilk false)
-      (outputformat 1)
+      (outputformat 4)
       (mirror false)
-      (drillshape 1)
+      (drillshape 0)
       (scaleselection 1)
-      (outputdirectory "")
+      (outputdirectory "../../")
     )
   )
@@
         (effects (font (size 1 1) (thickness 0.15)))
     )
-    (fp_text value "R" (at 0 1.43 90) (layer "F.Fab") hide
+    (fp_text value "33" (at 0 1.43 90) (layer "F.Fab") hide
         (effects (font (size 1 1) (thickness 0.15)))
     )
@@
         (effects (font (size 1 1) (thickness 0.15)))
     )
-    (fp_text value "Conn_01x02_Socket" (at 0 4.87) (layer "F.Fab") hide
+    (fp_text value "Conn_01x02_Pin" (at 0 4.87) (layer "F.Fab") hide
         (effects (font (size 1 1) (thickness 0.15)))
     )
@@
     (fp_line (start 3.6775 2.56) (end -3.6775 2.56)
       (stroke (width 0.1) (type solid)) (layer "F.Fab"))
-    (pad "1" smd roundrect (at -3.3875 0 90) (size 1.925 5.45) (layers "F.Cu" "F.Paste" "F.Mask") (roundrect_rratio 0.12987)
+    (pad "1" smd roundrect (at -3.3875 0 90) (size 1.925 5.45) (layers "F.Cu" "F.Paste" "F.Mask") (roundrect_rratio 0.1298701299)
       (net 68 "Net-(BT1-+)") (pintype "passive"))
-    (pad "2" smd roundrect (at 3.3875 0 90) (size 1.925 5.45) (layers "F.Cu" "F.Paste" "F.Mask") (roundrect_rratio 0.12987)
+    (pad "2" smd roundrect (at 3.3875 0 90) (size 1.925 5.45) (layers "F.Cu" "F.Paste" "F.Mask") (roundrect_rratio 0.1298701299)
       (net 1 "BATT_CONN") (pintype "passive"))
   )
